File: Hardware/power.kicad_sch (KiCad schematic)
At the start: 41 parts, among them IC1 LTC4413EDD#PBF, J3 XT30PW-M, Q1 SISS23DN-T1-GE3, Q5 SSM3K15AMFV,L3F, U3 LM66200DRLR, U4 MAX77827AEFD+T, U5 SC4215ASTRT

Commit message: V2 changes, post review work
Parts:
- added R27: 470k, Resistor_SMD:R_0402_1005Metric, symbol Device:R_Small
Connections:
- net +3V3: now also R27.1
- net ID_Stat: now also R27.2
Changed lines of the file:
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@@
 	)
 	(junction
+		(at 97.79 100.33)
+		(diameter 0)
+		(color 0 0 0 0)
+	)
+	(junction
 		(at 205.74 62.23)
 		(diameter 0)
@@
 	)
 	(junction
-		(at 114.3 102.87)
-		(diameter 0)
-		(color 0 0 0 0)
-	)
-	(junction
 		(at 143.51 146.05)
 		(diameter 0)
@@
 		)
 	)
-	(wire
-		(pts
-			(xy 93.98 97.79) (xy 114.3 97.79)
-		)
-		(stroke
-			(width 0)
-			(type default)
-		)
-	)
 	(polyline
 		(pts
@@
 	(wire
 		(pts
+			(xy 97.79 100.33) (xy 93.98 100.33)
+		)
+		(stroke
+			(width 0)
+			(type default)
+		)
+	)
+	(wire
+		(pts
 			(xy 254 62.23) (xy 254 63.5)
 		)
@@
 	(wire
 		(pts
+			(xy 97.79 97.79) (xy 97.79 100.33)
+		)
+		(stroke
+			(width 0)
+			(type default)
+		)
+	)
+	(wire
+		(pts
 			(xy 114.3 107.95) (xy 93.98 107.95)
 		)
@@
 	(wire
 		(pts
+			(xy 101.6 100.33) (xy 97.79 100.33)
+		)
+		(stroke
+			(width 0)
+			(type default)
+		)
+	)
+	(wire
+		(pts
 			(xy 27.94 97.79) (xy 40.64 97.79)
 		)
@@
 	(wire
 		(pts
-			(xy 114.3 97.79) (xy 114.3 102.87)
-		)
-		(stroke
-			(width 0)
-			(type default)
-		)
-	)
-	(wire
-		(pts
 			(xy 146.05 146.05) (xy 148.59 146.05)
 		)
@@
 	(wire
 		(pts
+			(xy 93.98 90.17) (xy 93.98 97.79)
+		)
+		(stroke
+			(width 0)
+			(type default)
+		)
+	)
+	(wire
+		(pts
 			(xy 151.13 171.45) (xy 151.13 175.26)
 		)
@@
 	)
 	(label "RBUS + Cell"
+		(at 93.98 90.17 180)
+		(effects
+			(font
+				(size 1.27 1.27)
+			)
+			(justify right bottom)
+		)
+	)
+	(label "RBUS + Cell"
 		(at 53.34 146.05 90)
 		(effects
@@
 	(hierarchical_label "ID_Stat"
 		(shape output)
-		(at 93.98 100.33 0)
+		(at 101.6 100.33 0)
 		(effects
 			(font
@@
 	)
 	(symbol
+		(lib_id "Device:R_Small")
+		(at 97.79 95.25 0)
+		(mirror y)
+		(unit 1)
+		(exclude_from_sim no)
+		(in_bom yes)
+		(on_board yes)
+		(dnp no)
+		(property "Reference" "R27"
+			(at 103.124 94.488 0)
+			(effects
+				(font
+					(size 1.27 1.27)
+				)
+				(justify left)
+			)
+		)
+		(property "Value" "470k"
+			(at 104.14 96.774 0)
+			(effects
+				(font
+					(size 1.27 1.27)
+				)
+				(justify left)
+			)
+		)
+		(property "Footprint" "Resistor_SMD:R_0402_1005Metric"
+			(at 97.79 95.25 0)
+			(effects
+				(font
+					(size 1.27 1.27)
+				)
+				(hide yes)
+			)
+		)
+		(property "Datasheet" "~"
+			(at 97.79 95.25 0)
+			(effects
+				(font
+					(size 1.27 1.27)
+				)
+				(hide yes)
+			)
+		)
+		(property "Description" ""
+			(at 97.79 95.25 0)
+			(effects
+				(font
+					(size 1.27 1.27)
+				)
+				(hide yes)
+			)
+		)
+		(pin "1"
+		)
+		(pin "2"
+		)
+		(instances
+			(project "Main board"
+				(path "/7db990e4-92e1-4f99-b4d2-435bbec1ba83/48a413b4-b7c2-44ac-971c-583c31b73475"
+					(reference "R27")
+					(unit 1)
+				)
+			)
+		)
+	)
+	(symbol
 		(lib_id "power:GND")
 		(at 200.66 67.31 0)
@@
 					(unit 1)
 				)
+			)
+		)
+	)
+	(symbol
+		(lib_id "power:+3.3V")
+		(at 97.79 92.71 0)
+		(unit 1)
+		(exclude_from_sim no)
+		(in_bom yes)
+		(on_board yes)
+		(dnp no)
+		(fields_autoplaced yes)
+		(property "Reference" "#PWR054"
+			(at 97.79 96.52 0)
+			(effects
+				(font
+					(size 1.27 1.27)
+				)
+				(hide yes)
+			)
+		)
+		(property "Value" "+3V3"
+			(at 97.79 89.1342 0)
+			(effects
+				(font
+					(size 1.27 1.27)
+				)
+			)
+		)
+		(property "Footprint" ""
+			(at 97.79 92.71 0)
+			(effects
+				(font
+					(size 1.27 1.27)
+				)
+				(hide yes)
+			)
+		)
+		(property "Datasheet" ""
+			(at 97.79 92.71 0)
+			(effects
+				(font
+					(size 1.27 1.27)
+				)
+				(hide yes)
+			)
+		)
+		(property "Description" ""
+			(at 97.79 92.71 0)
+			(effects
+				(font
+					(size 1.27 1.27)
+				)
+				(hide yes)
+			)
+		)
+		(pin "1"
+		)
+		(instances
+			(project "Main board"
+				(path "/7db990e4-92e1-4f99-b4d2-435bbec1ba83/48a413b4-b7c2-44ac-971c-583c31b73475"
+					(reference "#PWR054")
+					(unit 1)
+				)

Commit message: More V2 changes
Parts:
- R23: value 10k -> 120k
- R24: value 1.8k -> 18k
Other:
- note added: "Potential divider setup for minimal 3.3V on the RBUS logic, including potential variances of resistor values"
Changed lines of the file:
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@@
 		)
 	)
+	(text "Potential divider setup for minimal 3.3V on the RBUS logic,\nincluding potential variances of resistor values\n"
+		(exclude_from_sim no)
+		(at 45.974 89.154 0)
+		(effects
+			(font
+				(size 1.27 1.27)
+			)
+		)
+	)
 	(text "Be extra careful in leaving this connected at a single point\n"
 		(exclude_from_sim no)
@@
 			)
 		)
-		(property "Value" "10k"
+		(property "Value" "120k"
 			(at 85.4964 152.146 0)
 			(effects
@@
 			)
 		)
-		(property "Value" "1.8k"
+		(property "Value" "18k"
 			(at 85.4964 159.766 0)
 			(effects
