File: Hardware/Crosshair.kicad_sch (KiCad schematic)
At the start: 40 parts, among them U1 ESP32-S3, Y1 R940000171

Commit message: reformatted and renamed file
Parts:
- C103: renamed from C3; value 0.1uF -> 100nF
- C105: renamed from C5; value 0.1uF -> 100nF
- C106: renamed from C6; value 0.1uF -> 100nF
- C109: renamed from C8; value 0.1uF -> 100nF
- C110: renamed from C10; value 0.1uF -> 100nF
- C111: renamed from C11; value 0.1uF -> 100nF
- D101: renamed from TXLED1; value GREEN_LED -> LED_GREEN
- D102: renamed from CTXLED1; value GREEN_LED -> LED_GREEN
- D103: renamed from CRXLED1; value ORANGE_LED -> LED_ORANGE
- D104: renamed from 3V3LED1; value BLUE_LED -> LED_BLUE
- H101: renamed from H1; now left out of the parts list
- H102: renamed from H2; now left out of the parts list
- H103: renamed from H3; now left out of the parts list
- H104: renamed from H4; now left out of the parts list
- L101: renamed from L1; value 2.0nH -> 2nH
- R107: renamed from R6; value 499R -> 499Ω
- TP101: renamed from TP9; now left out of the parts list
- TP102: renamed from TP10; now left out of the parts list
- TP103: renamed from TP12; now left out of the parts list
- TP104: renamed from TP11; now left out of the parts list
- Y101: renamed from Y1; value R940000171 -> 40MHz±10ppm; MPN (none) -> R940000171
- renumbered C1 to C101, C2 to C102, C4 to C104, C7 to C107, C9 to C108, C13 to C112, C14 to C113, ENJUMPER1 to J101, BOOTJUMPER1 to J102, L2 to L102, R1 to R101, R2 to R102, R5 to R103, R18 to R104, R3 to R105, R4 to R106, R26 to R108, R29 to R109, U1 to U101
