File: Hardware/Crosshair.kicad_sch (KiCad schematic)
At the start: 40 parts, among them J101 Conn_01x02_Male, J102 Conn_01x02_Male, U101 ESP32-S3, Y101 40MHz±10ppm

Commit message: feat: Slight tweaks to filled zones, silkscreen, traces, and vias
Connections:
- net GPIO10 is gone; now on net GPIO9: U101.14 (GPIO9/ADC1_CH8)
- net GPIO7: now also U101.12 (GPIO7/ADC1_CH6); no longer U101.11 (GPIO6/ADC1_CH5)
- net GPIO8: now also U101.13 (GPIO8/ADC1_CH7); no longer U101.12 (GPIO7/ADC1_CH6)
- net GPIO9: no longer U101.13 (GPIO8/ADC1_CH7)
- new net GPIO6: U101.11 (GPIO6/ADC1_CH5)
Other:
- sheet GPIO ports: added GPIO6; removed GPIO10
Changed lines of the file:
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@@
 		)
 	)
-	(label "GPIO9"
+	(label "GPIO8"
 		(at 190.5 148.59 180)
 		(effects
@@
 		)
 	)
-	(label "GPIO7"
+	(label "GPIO6"
 		(at 190.5 143.51 180)
 		(effects
@@
 		)
 	)
-	(label "GPIO7"
+	(label "GPIO6"
 		(at 62.23 85.09 180)
 		(effects
@@
 		)
 	)
-	(label "GPIO10"
+	(label "GPIO9"
 		(at 62.23 92.71 180)
 		(effects
@@
 		)
 	)
-	(label "GPIO10"
+	(label "GPIO9"
 		(at 190.5 151.13 180)
 		(effects
@@
 		)
 	)
-	(label "GPIO8"
+	(label "GPIO7"
 		(at 190.5 146.05 180)
 		(effects
@@
 		)
 	)
-	(label "GPIO8"
+	(label "GPIO7"
 		(at 62.23 87.63 180)
 		(effects
@@
 		)
 	)
-	(label "GPIO9"
+	(label "GPIO8"
 		(at 62.23 90.17 180)
 		(effects
@@
 			)
 		)
-		(pin "GPIO9" bidirectional
+		(pin "GPIO8" bidirectional
 			(at 196.85 148.59 180)
 			(effects
@@
 			)
 		)
-		(pin "GPIO8" bidirectional
+		(pin "GPIO7" bidirectional
 			(at 196.85 146.05 180)
 			(effects
@@
 			)
 		)
-		(pin "GPIO10" bidirectional
+		(pin "GPIO9" bidirectional
 			(at 196.85 151.13 180)
 			(effects
@@
 			)
 		)
-		(pin "GPIO7" bidirectional
+		(pin "GPIO6" bidirectional
 			(at 196.85 143.51 180)
 			(effects
