File: Hardware/GPIO.kicad_sch (KiCad schematic)
At the start: 8 parts

Commit message: Extra tweaks - current sense etc
Connections:
- no-connect marks 0 -> 2
Changed lines of the file:
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@@
 		(color 0 0 0 0)
+	)
+	(no_connect
+		(at 137.16 80.01)
+	)
+	(no_connect
+		(at 106.68 80.01)
 	)
 	(wire
@@
 		)
 	)
-	(hierarchical_label "GPIO16"
-		(shape bidirectional)
-		(at 146.05 80.01 0)
-		(effects
-			(font
-				(size 1.27 1.27)
-			)
-			(justify left)
-		)
-	)
 	(hierarchical_label "GPIO7"
 		(shape bidirectional)
@@
 		(effects
 			(font
-				(size 1.27 1.27)
-			)
-			(justify right)
-		)
-	)
-	(hierarchical_label "GPIO15"
-		(shape bidirectional)
-		(at 101.6 80.01 180)
-		(effects
-			(font

Commit message: Mega commit
Post review changes
Parts:
- renumbered ENJUMPER4 to 3V3_GND1, ENJUMPER2 to GPIO_7/8, ENJUMPER3 to GPIO_9/10
Connections:
- net GPIO10: now also D6.3 (K/A_2); no longer D6.4 (K/A_3)
- net GPIO7: now also D6.1 (K/A_1); no longer D6.6 (K/A_5)
- net GPIO8: now also D6.5 (K/A_4); no longer D6.3 (K/A_2)
- net GPIO9: now also D6.6 (K/A_5); no longer D6.7 (K/A_6)
Changed lines of the file:
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@@
 	)
 	(no_connect
-		(at 137.16 80.01)
+		(at 137.16 85.09)
 	)
 	(no_connect
-		(at 106.68 80.01)
+		(at 106.68 87.63)
 	)
 	(wire
@@
 		)
 	)
+	(hierarchical_label "GPIO10"
+		(shape bidirectional)
+		(at 106.68 85.09 180)
+		(effects
+			(font
+				(size 1.27 1.27)
+			)
+			(justify right)
+		)
+	)
+	(hierarchical_label "GPIO9"
+		(shape bidirectional)
+		(at 137.16 82.55 0)
+		(effects
+			(font
+				(size 1.27 1.27)
+			)
+			(justify left)
+		)
+	)
 	(hierarchical_label "GPIO7"
 		(shape bidirectional)
@@
 		)
 	)
+	(hierarchical_label "GPIO9"
+		(shape bidirectional)
+		(at 143.51 125.73 270)
+		(effects
+			(font
+				(size 1.27 1.27)
+			)
+			(justify right)
+		)
+	)
+	(hierarchical_label "GPIO9"
+		(shape bidirectional)
+		(at 201.93 72.39 180)
+		(effects
+			(font
+				(size 1.27 1.27)
+			)
+			(justify right)
+		)
+	)
 	(hierarchical_label "GPIO8"
 		(shape bidirectional)
-		(at 106.68 85.09 180)
+		(at 149.86 125.73 270)
 		(effects
 			(font
@@
 	(hierarchical_label "GPIO7"
 		(shape bidirectional)
-		(at 137.16 82.55 0)
+		(at 106.68 80.01 180)
+		(effects
+			(font
+				(size 1.27 1.27)
+			)
+			(justify right)
+		)
+	)
+	(hierarchical_label "GPIO8"
+		(shape bidirectional)
+		(at 179.07 73.66 180)
+		(effects
+			(font
+				(size 1.27 1.27)
+			)
+			(justify right)
+		)
+	)
+	(hierarchical_label "GPIO10"
+		(shape bidirectional)
+		(at 201.93 74.93 180)
+		(effects
+			(font
+				(size 1.27 1.27)
+			)
+			(justify right)
+		)
+	)
+	(hierarchical_label "GPIO7"
+		(shape bidirectional)
+		(at 179.07 71.12 180)
+		(effects
+			(font
+				(size 1.27 1.27)
+			)
+			(justify right)
+		)
+	)
+	(hierarchical_label "GPIO8"
+		(shape bidirectional)
+		(at 137.16 80.01 0)
 		(effects
 			(font
@@
 			)
 			(justify left)
-		)
-	)
-	(hierarchical_label "GPIO9"
-		(shape bidirectional)
-		(at 143.51 125.73 270)
-		(effects
-			(font
-				(size 1.27 1.27)
-			)
-			(justify right)
-		)
-	)
-	(hierarchical_label "GPIO9"
-		(shape bidirectional)
-		(at 201.93 72.39 180)
-		(effects
-			(font
-				(size 1.27 1.27)
-			)
-			(justify right)
-		)
-	)
-	(hierarchical_label "GPIO8"
-		(shape bidirectional)
-		(at 149.86 125.73 270)
-		(effects
-			(font
-				(size 1.27 1.27)
-			)
-			(justify right)
-		)
-	)
-	(hierarchical_label "GPIO8"
-		(shape bidirectional)
-		(at 179.07 73.66 180)
-		(effects
-			(font
-				(size 1.27 1.27)
-			)
-			(justify right)
-		)
-	)
-	(hierarchical_label "GPIO10"
-		(shape bidirectional)
-		(at 201.93 74.93 180)
-		(effects
-			(font
-				(size 1.27 1.27)
-			)
-			(justify right)
-		)
-	)
-	(hierarchical_label "GPIO10"
-		(shape bidirectional)
-		(at 106.68 87.63 180)
-		(effects
-			(font
-				(size 1.27 1.27)
-			)
-			(justify right)
-		)
-	)
-	(hierarchical_label "GPIO9"
-		(shape bidirectional)
-		(at 137.16 85.09 0)
-		(effects
-			(font
-				(size 1.27 1.27)
-			)
-			(justify left)
-		)
-	)
-	(hierarchical_label "GPIO7"
-		(shape bidirectional)
-		(at 179.07 71.12 180)
-		(effects
-			(font
-				(size 1.27 1.27)
-			)
-			(justify right)
 		)
 	)
@@
 		(on_board yes)
 		(dnp no)
-		(property "Reference" "ENJUMPER2"
+		(property "Reference" "GPIO_7/8"
 			(at 185.42 67.31 90)
 			(effects
@@
 			(project "Main board"
 				(path "/7db990e4-92e1-4f99-b4d2-435bbec1ba83/4d7a61a6-e9d3-4ff3-bb3d-b277b97d3061"
-					(reference "ENJUMPER2")
+					(reference "GPIO_7/8")
 					(unit 1)
 				)
@@
 		(on_board yes)
 		(dnp no)
-		(property "Reference" "ENJUMPER3"
+		(property "Reference" "GPIO_9/10"
 			(at 208.28 68.58 90)
 			(effects
@@
 			(project "Main board"
 				(path "/7db990e4-92e1-4f99-b4d2-435bbec1ba83/4d7a61a6-e9d3-4ff3-bb3d-b277b97d3061"
-					(reference "ENJUMPER3")
+					(reference "GPIO_9/10")
 					(unit 1)
 				)
@@
 		(on_board yes)
 		(dnp no)
-		(property "Reference" "ENJUMPER4"
+		(property "Reference" "3V3_GND1"
 			(at 184.15 93.98 90)
 			(effects
@@
 			(project "Main board"
 				(path "/7db990e4-92e1-4f99-b4d2-435bbec1ba83/4d7a61a6-e9d3-4ff3-bb3d-b277b97d3061"
-					(reference "ENJUMPER4")
+					(reference "3V3_GND1")
 					(unit 1)
 				)

Commit message: reformatted and renamed file
Parts:
- R401: renamed from R30; value 10k -> 10kΩ
- R402: renamed from R31; value 10k -> 10kΩ
- R403: renamed from R32; value 10k -> 10kΩ
- R404: renamed from R33; value 10k -> 10kΩ
- renumbered D6 to D401, 3V3_GND1 to J401, GPIO_7/8 to J402, GPIO_9/10 to J403
