File: Hardware/GPIO.kicad_sch (KiCad schematic)
At the start: 8 parts, among them J401 Conn_01x02_Male, J402 Conn_01x02_Male, J403 Conn_01x02_Male

Commit message: feat: Slight tweaks to filled zones, silkscreen, traces, and vias
Connections:
- net GPIO10 is gone; now on net GPIO9: D401.3 (K/A_2), J403.1 (Pin_1), R404.2
- net GPIO7: now also D401.5 (K/A_4), J402.1 (Pin_1), R402.2; no longer D401.1 (K/A_1), J402.2 (Pin_2), R403.2
- net GPIO8: now also D401.6 (K/A_5), J403.2 (Pin_2), R401.2; no longer D401.5 (K/A_4), J402.1 (Pin_1), R402.2
- net GPIO9: no longer D401.6 (K/A_5), J403.2 (Pin_2), R401.2
- new net GPIO6: D401.1 (K/A_1), J402.2 (Pin_2), R403.2
Changed lines of the file:
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@@
 		)
 	)
-	(hierarchical_label "GPIO10"
+	(hierarchical_label "GPIO9"
 		(shape bidirectional)
 		(at 106.68 85.09 180)
@@
 		)
 	)
-	(hierarchical_label "GPIO9"
+	(hierarchical_label "GPIO8"
 		(shape bidirectional)
 		(at 137.16 82.55 0)
@@
 		)
 	)
-	(hierarchical_label "GPIO7"
+	(hierarchical_label "GPIO6"
 		(shape bidirectional)
 		(at 157.48 125.73 270)
@@
 		)
 	)
-	(hierarchical_label "GPIO9"
+	(hierarchical_label "GPIO8"
 		(shape bidirectional)
 		(at 143.51 125.73 270)
@@
 		)
 	)
-	(hierarchical_label "GPIO9"
+	(hierarchical_label "GPIO8"
 		(shape bidirectional)
 		(at 201.93 72.39 180)
@@
 		)
 	)
-	(hierarchical_label "GPIO8"
+	(hierarchical_label "GPIO7"
 		(shape bidirectional)
 		(at 149.86 125.73 270)
@@
 		)
 	)
-	(hierarchical_label "GPIO7"
+	(hierarchical_label "GPIO6"
 		(shape bidirectional)
 		(at 106.68 80.01 180)
@@
 		)
 	)
-	(hierarchical_label "GPIO8"
+	(hierarchical_label "GPIO7"
 		(shape bidirectional)
 		(at 179.07 73.66 180)
@@
 		)
 	)
-	(hierarchical_label "GPIO10"
+	(hierarchical_label "GPIO9"
 		(shape bidirectional)
 		(at 201.93 74.93 180)
@@
 		)
 	)
-	(hierarchical_label "GPIO7"
+	(hierarchical_label "GPIO6"
 		(shape bidirectional)
 		(at 179.07 71.12 180)
@@
 		)
 	)
-	(hierarchical_label "GPIO8"
+	(hierarchical_label "GPIO7"
 		(shape bidirectional)
 		(at 137.16 80.01 0)
@@
 		)
 	)
-	(hierarchical_label "GPIO10"
+	(hierarchical_label "GPIO9"
 		(shape bidirectional)
 		(at 165.1 125.73 270)
