File: Hardware/USB-RBUS.kicad_sch (KiCad schematic)
At the start: 5 parts, among them J4 USB_C_Receptacle_USB2.0

Commit message: reformatted and renamed file
Parts:
- D601: renamed from RBUSLED1; value WHITE_LED -> LED_WHITE
- TP601: renamed from TP3; now left out of the parts list
- TP602: renamed from TP7; now left out of the parts list
- renumbered J4 to J601, R25 to R601
