File: Hardware/Pyro.kicad_sch (KiCad schematic)
At the start: 11 parts, among them J5 7788, J6 7788, Q4 BSZ025N04LS, U12 TCMT1109

Commit message: reformatted and renamed file
Parts:
- D901: renamed from Firing1; value EMERALD_LED -> LED_GREEN
- D903: renamed from D4; value RED_LED -> LED_RED
- D904: renamed from D5; value 954-S-102T -> S-102T
- renumbered D3 to D902, J5 to J901, J6 to J902, Q4 to Q901, R39 to R901, R19 to R902, R20 to R903, U12 to U901

Commit message: changed 1 footprint
Parts:
- D904: footprint Diode_SMD:D_1206_3216Metric -> iclr:SODFL3516X70N
Changed lines of the file:
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@@
 			)
 		)
-		(property "Footprint" "Diode_SMD:D_1206_3216Metric"
+		(property "Footprint" "iclr:SODFL3516X70N"
 			(at 161.29 95.25 0)
 			(effects
