File: Hardware/Pyro.kicad_sch (KiCad schematic)
At the start: 11 parts, among them J901 7788, J902 7788, Q901 BSZ025N04LS, U901 TCMT1109

Commit message: feat: Changed BSZ025N04LS to BSZ024N04LS6, KiCad 10 save
Parts:
- Q901: value BSZ025N04LS -> BSZ024N04LS6
