File: Hardware/Crosshair.kicad_pcb (KiCad board)
At the start: 4 copper layers, 57.4 x 40 mm, 164 parts, among them J1001 DM3AT-SF-PEJM5_40_, J101 Conn_01x02_Male, J102 Conn_01x02_Male, J201 XT30PW-M, J401 Conn_01x02_Male, J402 Conn_01x02_Male, J403 Conn_01x02_Male, J501 USB_C_Receptacle_USB2.0, J601 USB_C_Receptacle_USB2.0, J901 7788, J902 7788, Q201 SISS23DN-T1-GE3, Q202 SSM3K15AMFV,L3F, Q301 BSZ025N04LS, Q302 BSZ025N04LS, Q901 BSZ025N04LS, U101 ESP32-S3, U201 LM66200DRLR, U202 LTC4413EDD#PBF, U203 MAX77827AEFD+T, U204 SC4215ASTRT, U301 TPS55288QRPMRQ1, U701 SN65HVD230, U801 DPS368, U901 TCMT1109, Y101 40MHz±10ppm

Commit message: feat: Slight tweaks to filled zones, silkscreen, traces, and vias
Parts:
- moved G*** 2.41 mm to (98.2, 77.0)
- moved R305 1.67 mm to (105.0, 98.8), turned to 180 degrees
- moved LED301 1.04 mm to (104.9, 97.5), turned to 180 degrees
- moved R503 0.83 mm to (138.1, 80.7)
Connections:
- D401 pad 1: /GPIO7 -> /GPIO6
- D401 pad 3: /GPIO10 -> /GPIO9
- D401 pad 5: /GPIO8 -> /GPIO7
- D401 pad 6: /GPIO9 -> /GPIO8
- J402 pad 1: /GPIO8 -> /GPIO7
- J402 pad 2: /GPIO7 -> /GPIO6
- J403 pad 1: /GPIO10 -> /GPIO9
- J403 pad 2: /GPIO9 -> /GPIO8
- R401 pad 2: /GPIO9 -> /GPIO8
- R402 pad 2: /GPIO8 -> /GPIO7
- R403 pad 2: /GPIO7 -> /GPIO6
- R404 pad 2: /GPIO10 -> /GPIO9
- U101 pad 11: /GPIO7 -> /GPIO6
- U101 pad 12: /GPIO8 -> /GPIO7
- U101 pad 13: /GPIO9 -> /GPIO8
- U101 pad 14: /GPIO10 -> /GPIO9
Routing:
- net /GPIO6: track 0.00 -> 11.0 mm
- net /GPIO10: track 9.96 -> 0.00 mm
- net /GPIO8: track 11.5 -> 8.61 mm
- net GND: track 199.8 -> 198.1 mm, vias 298 -> 300
- net /GPIO9: track 8.61 -> 9.96 mm
- net VBUS: track 55.2 -> 54.1 mm
- added copper zone on In2.Cu, net GND

Commit message: feat: Changed BSZ025N04LS to BSZ024N04LS6, KiCad 10 save
Parts:
- Q301, Q302, Q901: value BSZ025N04LS -> BSZ024N04LS6
