File: Hardware/Volt_reg.kicad_sch (KiCad schematic)
At the start: 27 parts, among them Q301 BSZ025N04LS, Q302 BSZ025N04LS, U301 TPS55288QRPMRQ1

Commit message: feat: Changed BSZ025N04LS to BSZ024N04LS6, KiCad 10 save
Parts:
- Q301, Q302: value BSZ025N04LS -> BSZ024N04LS6
